Commit message: fix(sirius_gazebo): Use correct variable (gazebo_origin) in gnss macro

File: sirius_description/urdf/sirius/gnss.urdf.xacro (robot description, xacro)
@@ -3,5 +3,5 @@
      https://www.sparkfun.com/products/21801 -->
 <robot xmlns:xacro="http://wiki.ros.org/xacro">
-<xacro:macro name="gnss" params="prefix:='' material collisions:=${xacro.load_yaml('$(find sirius_description)/urdf/sirius/collisions.yaml')} datum:=^ elevation:=^ horizontal_cep:=1.0 vertical_cep:=1.5 rate:=20.0 spawn_origin:=^">
+<xacro:macro name="gnss" params="prefix:='' material collisions:=${xacro.load_yaml('$(find sirius_description)/urdf/sirius/collisions.yaml')} datum:=^ elevation:=^ horizontal_cep:=1.0 vertical_cep:=1.5 rate:=20.0 gazebo_origin:=^">
   <xacro:property name="_prefix" value="${prefix + '_' if prefix else ''}"/>
   <!-- sqrt(-1/(2*ln(0.5))) = 0.8493218002880191 -->
@@ -67,5 +67,5 @@
         </sphericalCoordinates>
         <!-- <positionCovariance>${horizontal_stddev} 0 0 0 ${horizontal_stddev} 0 0 0 ${vertical_stddev}</positionCovariance> -->
-        <spawnOrigin>${spawn_origin[0]} ${spawn_origin[1]}</spawnOrigin>
+        <gazeboOrigin>${gazebo_origin[0]} ${gazebo_origin[1]}</gazeboOrigin>
       </plugin>
     </sensor>

Commit message: feat: move base flex tests

File: sirius_description/urdf/sirius/gnss.urdf.xacro (robot description, xacro)
@@ -3,5 +3,5 @@
      https://www.sparkfun.com/products/21801 -->
 <robot xmlns:xacro="http://wiki.ros.org/xacro">
-<xacro:macro name="gnss" params="prefix:='' material collisions:=${xacro.load_yaml('$(find sirius_description)/urdf/sirius/collisions.yaml')} datum:=^ elevation:=^ horizontal_cep:=1.0 vertical_cep:=1.5 rate:=20.0 gazebo_origin:=^">
+<xacro:macro name="gnss" params="prefix:='' material collisions:=${xacro.load_yaml('$(find sirius_description)/urdf/sirius/collisions.yaml')} datum:=^ elevation:=^ horizontal_cep:=0.01443 vertical_cep:=0.02886 rate:=20.0 gazebo_origin:=^">
   <xacro:property name="_prefix" value="${prefix + '_' if prefix else ''}"/>
   <!-- sqrt(-1/(2*ln(0.5))) = 0.8493218002880191 -->
