Commit message: feat: Manip visualization including 6th dof

File: sirius_description/urdf/oak-d-w/oak-d-w.urdf.xacro (robot description, xacro)
@@ -1,5 +1,5 @@
 <?xml version="1.0"?>
 <robot xmlns:xacro="http://ros.org/wiki/xacro">
-<xacro:macro name="oak-d-w" params="prefix:=oak-d-w collisions:=${xacro.load_yaml('$(find sirius_description)/urdf/oak-d-w/collisions.yaml')} stereo_fps:=^|30 imu_frequency:=^|200 datum:=^ elevation:=^ year:=^ calibration:=${xacro.load_yaml('$(find sirius_calibration)/kalibr/camimu/inflated/camimu-camchain-imucam.yaml')} imu_calibration:=${xacro.load_yaml('$(find sirius_calibration)/kalibr/camimu/inflated/camimu-imu.yaml')}">
+<xacro:macro name="oak-d-w" params="prefix:=oak-d-w collisions:=${xacro.load_yaml('$(find sirius_description)/urdf/oak-d-w/collisions.yaml')} stereo_fps:=^|30 imu_frequency:=^|200  calibration:=${xacro.load_yaml('$(find sirius_calibration)/kalibr/camimu/inflated/camimu-camchain-imucam.yaml')} imu_calibration:=${xacro.load_yaml('$(find sirius_calibration)/kalibr/camimu/inflated/camimu-imu.yaml')}">
   <xacro:property name="optical_offset_x" value="-0.01" />
   <xacro:property name="baseline" value="${sqrt(calibration.cam1.T_cn_cnm1[0][3]**2 + calibration.cam1.T_cn_cnm1[1][3]**2 + calibration.cam1.T_cn_cnm1[2][3]**2)}"/>
@@ -196,108 +196,4 @@
     </sensor>
   </gazebo>
-  <!-- IMU -->
-  <gazebo reference="${prefix}_camera_imu_link">
-    <sensor type="imu" name="imu_sensor">
-      <always_on>true</always_on>
-      <update_rate>${imu_frequency}</update_rate>
-      <imu>
-        <angular_velocity>
-          <x>
-            <noise type="gaussian">
-              <stddev>${gyroscope_stddev}</stddev>
-              <bias_stddev>${gyroscope_bias_stddev}</bias_stddev>
-            </noise>
-          </x>
-          <y>
-            <noise type="gaussian">
-              <stddev>${gyroscope_stddev}</stddev>
-              <bias_stddev>${gyroscope_bias_stddev}</bias_stddev>
-            </noise>
-          </y>
-          <z>
-            <noise type="gaussian">
-              <stddev>${gyroscope_stddev}</stddev>
-              <bias_stddev>${gyroscope_bias_stddev}</bias_stddev>
-            </noise>
-          </z>
-        </angular_velocity>
-        <linear_acceleration>
-          <x>
-            <noise type="gaussian">
-              <stddev>${accelerometer_stddev}</stddev>
-              <bias_stddev>${accelerometer_bias_stddev}</bias_stddev>
-            </noise>
-          </x>
-          <y>
-            <noise type="gaussian">
-              <stddev>${accelerometer_stddev}</stddev>
-              <bias_stddev>${accelerometer_bias_stddev}</bias_stddev>
-            </noise>
-          </y>
-          <z>
-            <noise type="gaussian">
-              <stddev>${accelerometer_stddev}</stddev>
-              <bias_stddev>${accelerometer_bias_stddev}</bias_stddev>
-            </noise>
-          </z>
-        </linear_acceleration>
-      </imu>
-      <plugin filename="libsirius_gazebo_ros_imu_sensor.so" name="imu_plugin">
-        <topicName>/${prefix}_camera/imu/data</topicName>
-        <frameName>${prefix}_camera_imu_link</frameName>
-        <updateRateHZ>${imu_frequency}</updateRateHZ>
-        <initialOrientationAsReference>false</initialOrientationAsReference>
-        <xyzOffset>0 0.0 0.0</xyzOffset>
-        <rpyOffset>0 0 ${datum[2] * pi/180}</rpyOffset>
-        <orientationCovariance>0.061086523819801536 0.061086523819801536 0.061086523819801536</orientationCovariance> <!-- 3.5deg from datasheet -->
-        <angularVelocityCovariance>${gyroscope_stddev**2} ${gyroscope_stddev**2} ${gyroscope_stddev**2}</angularVelocityCovariance>
-        <linearAccelerationCovariance>${100*accelerometer_stddev**2} ${100*accelerometer_stddev**2} ${100*accelerometer_stddev**2}</linearAccelerationCovariance>
-      </plugin>
-    </sensor>
-  </gazebo>
-  <!-- MAGNETOMETER -->
-  <gazebo reference="${prefix}_camera_imu_link">
-    <sensor type="magnetometer" name="magnetometer_sensor">
-      <always_on>true</always_on>
-        <!-- In practice, the magnetometer runs slower than the IMU, but
-        hardware fusion handles this and provides orientation at high rate.
-        In simulation, we use software fusion from imu_tools which uses
-        synchronizer that will drop imu messages if magnetometer runs at
-        slower rate. -->
-        <updateRateHZ>${imu_frequency}</updateRateHZ>
-      <magnetometer>
-        <!-- Noise parameters are taken from the datasheet -->
-        <!-- Datasheet: https://www.bosch-sensortec.com/media/boschsensortec/downloads/datasheets/bst-bmf055-ds000.pdf -->
-        <!-- "Output Noise" for worst case is used -->
-        <x>
-          <noise type="gaussian">
-            <stddev>1.4e-6</stddev>
-          </noise>
-        </x>
-        <y>
-          <noise type="gaussian">
-            <stddev>1.4e-6</stddev>
-          </noise>
-        </y>
-        <z>
-          <noise type="gaussian">
-            <stddev>1.4e-6</stddev>
-          </noise>
-        </z>
-      </magnetometer>
-      <plugin filename="libsirius_gazebo_ros_magnetometer_sensor.so" name="magnetometer_plugin">
-        <topicName>/${prefix}_camera/imu/mag</topicName>
-        <frameName>${prefix}_camera_imu_link</frameName>
-        <updateRateHZ>${imu_frequency}</updateRateHZ>
-        <sphericalCoordinates>
-          <latitudeDeg>${datum[0]}</latitudeDeg>
-          <longitudeDeg>${datum[1]}</longitudeDeg>
-          <headingDeg>${datum[2]}</headingDeg>
-          <elevation>${elevation}</elevation>
-          <year>${year}</year>
-        </sphericalCoordinates>
-      </plugin>
-    </sensor>
-  </gazebo>
   <gazebo reference="${prefix}_camera">
       <visual>

File: sirius_description/urdf/sirius/manipulator.urdf.xacro (robot description, xacro)
@@ -2,108 +2,249 @@
 <robot xmlns:xacro="http://www.ros.org/wiki/xacro" name="manipulator">
   <xacro:property name="package" value="sirius_description" />
-  <xacro:property name="base_length" value="0.006" />
-  <xacro:property name="cyl_length" value="0.0655" />
-  <xacro:property name="arm1_length" value="0.43498" />
-  <xacro:property name="arm2_length" value="0.5236" />
-  <xacro:property name="arm2_lever" value="0.0586" />
-  <xacro:property name="arm3_length" value="0.129" />
-  <xacro:property name="tool_length" value="0.18" />
-  <xacro:property name="base_size_x" value="0.2" />
-  <xacro:property name="arm1_home_angle" value="-0.7853981633974483"/>
-  <xacro:property name="arm2_home_angle" value="2.356194490192345"/>
-  <xacro:property name="arm3_home_angle" value="0.5"/>
-  <link name="root_link">
-  </link>
-  <joint name="root_base" type="fixed">
-    <parent link="root_link"/>
-    <child link="base_link"/>
-  </joint>
-  <link name="base_link">
-    <visual>
-      <origin xyz="0 0 0" rpy="0 0 0" />
+  <!-- Parse parameters -->
+  <!-- Load model parameters -->
+  <xacro:property name="params" value="${xacro.load_yaml('manipulator.yaml')}" />
+  <!-- Load inertial parameters -->
+  <xacro:property name="inertial" value="${xacro.load_yaml('manipulator_inertial.yaml')}" />
+  <xacro:include filename="$(find sirius_description)/urdf/oak-d-w/oak-d-w.urdf.xacro" />
+  <!-- Macro to simplify joint definition -->
+  <xacro:macro name="joint" params="type:='fixed' parent:='base_link' child:='' xyz:='0 0 0' rpy:='0 0 0' axis:='0 0 1' limit_effort:='0.0' limit_velocity:='0.0'">
+    <joint name="${child}_joint" type="${type}">
+      <parent link="${parent}"/>
+      <child link="${child}"/>
+      <origin xyz="${xyz}" rpy="${rpy}"/>
+      <axis xyz="${axis}"/>
+      <xacro:if value="${type != 'fixed'}">
+        <limit effort="${limit_effort}" velocity="${limit_velocity}"/>
+      </xacro:if>
+    </joint>
+  </xacro:macro>
+  <link name="manip_base_link">
+    <visual>
       <geometry>
         <mesh filename="package://${package}/meshes/manipulator/base.stl" scale="0.001 0.001 0.001"/>
       </geometry>
-    </visual>
-  </link>
+      <material name="grey">
+        <color rgba=".5 .5 .5 1" />
+      </material>
+    </visual>
+    <!-- <inertial>
+      <mass value="${inertial['base_mass']}"/>
+      <inertia ixx="${inertial['base_inertia']['ixx']}" ixy="${inertial['base_inertia']['ixy']}" ixz="${inertial['base_inertia']['ixz']}" iyy="${inertial['base_inertia']['iyy']}" iyz="${inertial['base_inertia']['iyz']}" izz="${inertial['base_inertia']['izz']}"/>
+    </inertial> -->
+    <collision>
+      <origin xyz="0 0 ${params['base_length'] / 2}" rpy="0 0 0" />
+      <geometry>
+        <box size="0.192 0.337 ${params['base_length']}" />
+      </geometry>
+    </collision>
+  </link>
+  <gazebo reference="manip_base_link">
+    <material>
+                                Gazebo/Grey
+    </material>
+  </gazebo>
+  <link name="cylinder">
+    <visual>
+      <origin xyz="0 0 0" rpy="0 0 0" />
+      <geometry>
+        <mesh filename="package://${package}/meshes/manipulator/cyl.stl" scale="0.001 0.001 0.001"/>
+      </geometry>
+      <material name="grey">
+      </material>
+    </visual>
+    <inertial>
+      <mass value="${inertial['cyl_mass']}"/>
+      <inertia ixx="${inertial['cyl_inertia']['ixx']}" ixy="${inertial['cyl_inertia']['ixy']}" ixz="${inertial['cyl_inertia']['ixz']}" iyy="${inertial['cyl_inertia']['iyy']}" iyz="${inertial['cyl_inertia']['iyz']}" izz="${inertial['cyl_inertia']['izz']}"/>
+    </inertial>
+    <collision>
+      <origin xyz="0 0 ${params['cyl_length']/2}" rpy="0 0 0" />
+      <geometry>
+        <cylinder length="${params['cyl_length']}" radius="0.06" />
+      </geometry>
+    </collision>
+  </link>
+  <gazebo reference="cylinder">
+    <material>
+                                Gazebo/Grey
+    </material>
+  </gazebo>
   <joint name="waist" type="continuous">
-    <parent link="base_link"/>
+    <parent link="manip_base_link"/>
     <child link="cylinder"/>
-    <origin xyz="0 0 ${base_length}"/>
+    <origin xyz="0 0 ${params['base_length']}"/>
     <axis xyz="0 0 1"/>
-  </joint>
-  <link name="cylinder">
-    <visual>
-      <origin xyz="0 0 0" rpy="0 0 0" />
-      <geometry>
-        <mesh filename="package://${package}/meshes/manipulator/cyl.stl" scale="0.001 0.001 0.001"/>
-      </geometry>
-    </visual>
-  </link>
+    <limit effort="100" velocity="5" />
+  </joint>
+  <transmission name="trans_base_cyl">
+    <type>transmission_interface/SimpleTransmission</type>
+    <joint name="waist">
+      <hardwareInterface>hardware_interface/VelocityJointInterface</hardwareInterface>
+    </joint>
+    <actuator name="motor_base_cyl">
+      <hardwareInterface>hardware_interface/VelocityJointInterface</hardwareInterface>
+      <mechanicalReduction>150</mechanicalReduction>
+    </actuator>
+  </transmission>
+  <link name="arm1">
+    <visual>
+      <origin xyz="0 0 0" rpy="0 0 0" />
+      <geometry>
+        <mesh filename="package://${package}/meshes/manipulator/arm1.stl" scale="0.001 0.001 0.001"/>
+      </geometry>
+      <material name="white">
+        <color rgba="1 1 1 1" />
+      </material>
+    </visual>
+    <inertial>
+      <mass value="${inertial['arm1_mass']}"/>
+      <inertia ixx="${inertial['arm1_inertia']['ixx']}" ixy="${inertial['arm1_inertia']['ixy']}" ixz="${inertial['arm1_inertia']['ixz']}" iyy="${inertial['arm1_inertia']['iyy']}" iyz="${inertial['arm1_inertia']['iyz']}" izz="${inertial['arm1_inertia']['izz']}"/>
+    </inertial>
+    <collision>
+      <origin xyz="0 0 ${params['arm1_length']/2}" rpy="0 0 0" />
+      <geometry>
+        <box size="0.07 0.07 ${params['arm1_length']}" />
+      </geometry>
+    </collision>
+  </link>
+  <gazebo reference="arm1">
+    <material>
+                                Gazebo/White
+    </material>
+  </gazebo>
   <joint name="shoulder" type="revolute">
     <parent link="cylinder"/>
     <child link="arm1"/>
-    <origin xyz="0 0 ${cyl_length}" rpy="0 ${arm1_home_angle} 0"/>
+    <origin xyz="0 0 ${params['cyl_length']}" rpy="0 ${params['arm1_home_angle']} 0"/>
     <axis xyz="0 1 0"/>
-    <limit
-      lower="${-1.45 - arm1_home_angle}"
-      upper="${1.45 - arm1_home_angle}"
-      effort="10"
-      velocity="5" />
-  </joint>
-  <link name="arm1">
-    <visual>
-      <origin xyz="0 0 0" rpy="0 0 0" />
-      <geometry>
-        <mesh filename="package://${package}/meshes/manipulator/arm1.stl" scale="0.001 0.001 0.001"/>
-      </geometry>
-    </visual>
-  </link>
+    <limit lower="${-1.45 - params['arm1_home_angle']}" upper="${1.45 - params['arm1_home_angle']}" effort="10" velocity="5" />
+  </joint>
+  <transmission name="trans_cyl_arm1">
+    <type>transmission_interface/SimpleTransmission</type>
+    <joint name="shoulder">
+      <hardwareInterface>hardware_interface/VelocityJointInterface</hardwareInterface>
+    </joint>
+    <actuator name="motor_cyl_arm1">
+      <hardwareInterface>hardware_interface/VelocityJointInterface</hardwareInterface>
+      <mechanicalReduction>120</mechanicalReduction>
+    </actuator>
+  </transmission>
+  <link name="arm2">
+    <visual>
+      <origin xyz="0 0 0" rpy="0 0 0" />
+      <geometry>
+        <mesh filename="package://${package}/meshes/manipulator/arm2.stl" scale="0.001 0.001 0.001"/>
+      </geometry>
+      <material name="grey">
+      </material>
+    </visual>
+    <inertial>
+      <mass value="${inertial['arm2_mass']}"/>
+      <inertia ixx="${inertial['arm2_inertia']['ixx']}" ixy="${inertial['arm2_inertia']['ixy']}" ixz="${inertial['arm2_inertia']['ixz']}" iyy="${inertial['arm2_inertia']['iyy']}" iyz="${inertial['arm2_inertia']['iyz']}" izz="${inertial['arm2_inertia']['izz']}"/>
+    </inertial>
+    <collision>
+      <origin xyz="0 0 ${params['arm2_length']/2 - params['arm2_lever']}" rpy="0 0 0" />
+      <geometry>
+        <box size="0.06 0.06 ${params['arm2_length']}" />
+      </geometry>
+    </collision>
+  </link>
+  <gazebo reference="arm2">
+    <material>
+                                Gazebo/Grey
+    </material>
+  </gazebo>
   <joint name="elbow" type="revolute">
     <parent link="arm1"/>
     <child link="arm2"/>
-    <origin xyz="0 0 ${arm1_length}" rpy="0 ${arm2_home_angle} 0"/>
+    <origin xyz="0 0 ${params['arm1_length']}" rpy="0 ${params['arm2_home_angle']} 0"/>
     <axis xyz="0 1 0"/>
-    <limit
-      lower="-1.6"
-      upper="0.0"
-      effort="100"
-      velocity="50" />
-  </joint>
-  <link name="arm2">
-    <visual>
-      <origin xyz="0 0 0" rpy="0 0 0" />
-      <geometry>
-        <mesh filename="package://${package}/meshes/manipulator/arm2.stl" scale="0.001 0.001 0.001"/>
-      </geometry>
-    </visual>
-  </link>
+    <limit lower="-1.6" upper="0.0" effort="100" velocity="50" />
+  </joint>
+  <transmission name="trans_elbow">
+    <type>transmission_interface/SimpleTransmission</type>
+    <joint name="elbow">
+      <hardwareInterface>hardware_interface/VelocityJointInterface</hardwareInterface>
+    </joint>
+    <actuator name="motor_elbow">
+      <hardwareInterface>hardware_interface/VelocityJointInterface</hardwareInterface>
+      <mechanicalReduction>100</mechanicalReduction>
+    </actuator>
+  </transmission>
+  <link name="arm3">
+    <visual>
+      <origin xyz="0 0 0" rpy="0 0 0" />
+      <geometry>
+        <mesh filename="package://${package}/meshes/manipulator/arm3.stl" scale="0.001 0.001 0.001"/>
+      </geometry>
+      <material name="white">
+      </material>
+    </visual>
+    <inertial>
+      <mass value="${inertial['arm3_mass']}"/>
+      <inertia ixx="${inertial['arm3_inertia']['ixx']}" ixy="${inertial['arm3_inertia']['ixy']}" ixz="${inertial['arm3_inertia']['ixz']}" iyy="${inertial['arm3_inertia']['iyy']}" iyz="${inertial['arm3_inertia']['iyz']}" izz="${inertial['arm3_inertia']['izz']}"/>
+    </inertial>
+    <collision>
+      <origin xyz="0 0 ${params['arm3_length']/2}" rpy="0 0 0" />
+      <geometry>
+        <box size="0.06 0.076 ${params['arm3_length']}" />
+      </geometry>
+    </collision>
+  </link>
+  <gazebo reference="arm3">
+    <material>
+                                Gazebo/White
+    </material>
+  </gazebo>
   <joint name="wrist_lift" type="revolute">
     <parent link="arm2"/>
     <child link="arm3"/>
-    <origin xyz="0 0 ${arm2_length - arm2_lever}" rpy="0 ${arm3_home_angle} 0"/>
+    <origin xyz="0 0 ${params['arm2_length'] - params['arm2_lever']}" rpy="0 ${params['arm3_home_angle']} 0"/>
     <axis xyz="0 1 0"/>
-    <limit
-      lower="-1.57"
-      upper="0"
-      effort="100"
-      velocity="50" />
-  </joint>
-  <link name="arm3">
-    <visual>
-      <origin xyz="0 0 0" rpy="0 0 0" />
-      <geometry>
-        <mesh filename="package://${package}/meshes/manipulator/arm3.stl" scale="0.001 0.001 0.001"/>
-      </geometry>
-    </visual>
+    <limit lower="-1.57" upper="0" effort="100" velocity="50" />
+  </joint>
+  <transmission name="trans_wrist_lift">
+    <type>transmission_interface/SimpleTransmission</type>
+    <joint name="wrist_lift">
+      <hardwareInterface>hardware_interface/VelocityJointInterface</hardwareInterface>
+    </joint>
+    <actuator name="motor_wrist_lift">
+      <hardwareInterface>hardware_interface/VelocityJointInterface</hardwareInterface>
+      <mechanicalReduction>1</mechanicalReduction>
+    </actuator>
+  </transmission>
+  <link name="fake">
   </link>
   <joint name="wrist_turn" type="continuous">
     <parent link="arm3"/>
     <child link="fake"/>
-    <origin xyz="0 0 ${arm3_length}"/>
+    <origin xyz="0 0 ${params['arm3_length']}"/>
     <axis xyz="1 0 0"/>
   </joint>
-  <link name="fake">
-  </link>
+  <link name="tool">
+    <visual>
+      <origin xyz="0 0 0" rpy="0 0 0" />
+      <geometry>
+        <mesh filename="package://${package}/meshes/manipulator/tool.stl" scale="0.001 0.001 0.001"/>
+      </geometry>
+      <material name="grey">
+      </material>
+    </visual>
+    <inertial>
+      <mass value="${inertial['tool_mass']}"/>
+      <inertia ixx="${inertial['tool_inertia']['ixx']}" ixy="${inertial['tool_inertia']['ixy']}" ixz="${inertial['tool_inertia']['ixz']}" iyy="${inertial['tool_inertia']['iyy']}" iyz="${inertial['tool_inertia']['iyz']}" izz="${inertial['tool_inertia']['izz']}"/>
+    </inertial>
+    <collision>
+      <origin xyz="0 0 ${params['tool_length']/2}" rpy="0 0 0" />
+      <geometry>
+        <cylinder length="${params['tool_length']}" radius="0.03" />
+      </geometry>
+    </collision>
+  </link>
+  <gazebo reference="tool">
+    <material>
+                                Gazebo/Grey
+    </material>
+  </gazebo>
   <joint name="wrist_spin" type="continuous">
     <parent link="fake"/>
@@ -111,19 +252,28 @@
     <origin xyz="0 0 0"/>
     <axis xyz="0 0 1"/>
-  </joint>
-  <link name="tool">
-    <visual>
-      <origin xyz="0 0 0" rpy="0 0 0" />
-      <geometry>
-        <mesh filename="package://${package}/meshes/manipulator/tool.stl" scale="0.001 0.001 0.001"/>
-      </geometry>
-    </visual>
-  </link>
+    <limit effort="20" velocity="5" />
+  </joint>
+  <transmission name="trans_wrist_spin">
+    <type>transmission_interface/SimpleTransmission</type>
+    <joint name="wrist_spin">
+      <hardwareInterface>hardware_interface/VelocityJointInterface</hardwareInterface>
+    </joint>
+    <actuator name="motor_wrist_spin">
+      <hardwareInterface>hardware_interface/VelocityJointInterface</hardwareInterface>
+      <mechanicalReduction>1</mechanicalReduction>
+    </actuator>
+  </transmission>
   <link name="virtual">
   </link>
-    <joint name="tool_virtual" type="fixed">
-      <parent link="tool"/>
-      <child link="virtual"/>
-      <origin xyz="0 0 ${tool_length}"/>
-    </joint>
+  <joint name="tool_virtual" type="fixed">
+    <parent link="tool"/>
+    <child link="virtual"/>
+    <origin xyz="0 0 ${params['tool_length']}"/>
+  </joint>
+  <gazebo>
+    <plugin name="gazebo_ros_control" filename="libgazebo_ros_control.so">
+      <robotNamespace>manipulator</robotNamespace>
+      <robotSimType>gazebo_ros_control/DefaultRobotHWSim</robotSimType>
+    </plugin>
+  </gazebo>
 </robot>
