Commit message: Added option to display manipulator

File: sirius_description/robots/sirius.urdf (robot description, URDF)
Before this commit: robot sirius, 30 links, 29 joints
Links:
- added link arm1; visual mesh filename=package://sirius_description/meshes/manipulator/arm1.stl scale=0.001 0.001 0.001
- added link arm2; visual mesh filename=package://sirius_description/meshes/manipulator/arm2.stl scale=0.001 0.001 0.001
- added link arm3; visual mesh filename=package://sirius_description/meshes/manipulator/arm3.stl scale=0.001 0.001 0.001
- added link cylinder; visual mesh filename=package://sirius_description/meshes/manipulator/cyl.stl scale=0.001 0.001 0.001
- added link fake
- added link manipulator_base_link; visual mesh filename=package://sirius_description/meshes/manipulator/base.stl scale=0.001 0.001 0.001
- added link root_link
- added link tool; visual mesh filename=package://sirius_description/meshes/manipulator/tool.stl scale=0.001 0.001 0.001
- added link virtual
Joints:
- added joint elbow: type revolute, parent arm1, child arm2, origin xyz=0 0 0.43498 rpy=0 2.356194490192345 0, axis 0 1 0, limit lower=-1.6 upper=0.0 effort=100 velocity=50
- added joint root_base: type fixed, parent root_link, child manipulator_base_link
- added joint shoulder: type revolute, parent cylinder, child arm1, origin xyz=0 0 0.0655 rpy=0 -0.7853981633974483 0, axis 0 1 0, limit lower=-0.6646018366025517 upper=2.2353981633974485 effort=10 velocity=5
- added joint tool_virtual: type fixed, parent tool, child virtual, origin xyz=0 0 0.18
- added joint waist: type continuous, parent manipulator_base_link, child cylinder, origin xyz=0 0 0.006, axis 0 0 1
- added joint wrist_lift: type revolute, parent arm2, child arm3, origin xyz=0 0 0.46499999999999997 rpy=0 0.5 0, axis 0 1 0, limit lower=-1.57 upper=0 effort=100 velocity=50
- added joint wrist_spin: type continuous, parent fake, child tool, origin xyz=0 0 0, axis 0 0 1
- added joint wrist_turn: type continuous, parent arm3, child fake, origin xyz=0 0 0.129, axis 1 0 0

File: sirius_description/robots/sirius.urdf.xacro (robot description, xacro)
@@ -8,4 +8,5 @@
   <xacro:arg name="stereo_fps" default="30"/>
   <xacro:arg name="year" default=""/>
+  <xacro:arg name="manipulator" default="5DOF"/>
   <xacro:property name="calibration_path" value="$(arg calibration_path)" />
   <xacro:if value="${calibration_path != ''}">
@@ -18,4 +19,5 @@
   <xacro:property name="stereo_fps" value="$(arg stereo_fps)" />
   <xacro:property name="year" value="$(arg year)" />
+  <xacro:property name="manipulator" value="$(arg manipulator)"/>
   <!-- Load model parameters -->
   <xacro:property name="mechanical" value="${xacro.load_yaml('$(find sirius_description)/config/mechanical.yaml')}" />
@@ -93,4 +95,8 @@
     <xacro:wheel_interface name="front_right" />
   </ros2_control>
+  <xacro:if value="${manipulator != ''}">
+    <xacro:include filename="$(find sirius_description)/urdf/sirius/manipulators/$(arg manipulator).urdf.xacro" />
+    <xacro:joint parent="platform" child="root_link" xyz="${mechanical['suspension_separation_x']/2} 0 ${mechanical['suspension_z'] + 0.045}" rpy="0 0 0"/>
+  </xacro:if>
   <gazebo>
     <plugin filename="libgazebo_ros2_control.so" name="gazebo_ros2_control">

File: sirius_description/urdf/sirius/manipulators/5DOF.urdf.xacro (robot description, xacro)
@@ -1,4 +1,4 @@
 <?xml version="1.0" encoding="utf-8"?>
-<robot xmlns:xacro="http://www.ros.org/wiki/xacro" name="manipulator">
+<robot xmlns:xacro="http://www.ros.org/wiki/xacro" name="5DOF">
   <xacro:property name="package" value="sirius_description" />
   <xacro:property name="base_length" value="0.006" />
@@ -17,16 +17,16 @@
   <joint name="root_base" type="fixed">
     <parent link="root_link"/>
-    <child link="base_link"/>
+    <child link="manipulator_base_link"/>
   </joint>
-  <link name="base_link">
+  <link name="manipulator_base_link">
     <visual>
       <origin xyz="0 0 0" rpy="0 0 0" />
       <geometry>
-        <mesh filename="package://${package}/meshes/manipulator/base.stl" scale="0.001 0.001 0.001"/>
+        <mesh filename="package://${package}/meshes/manipulators/5DOF/base.stl" scale="0.001 0.001 0.001"/>
       </geometry>
     </visual>
   </link>
   <joint name="waist" type="continuous">
-    <parent link="base_link"/>
+    <parent link="manipulator_base_link"/>
     <child link="cylinder"/>
     <origin xyz="0 0 ${base_length}"/>
@@ -37,5 +37,5 @@
       <origin xyz="0 0 0" rpy="0 0 0" />
       <geometry>
-        <mesh filename="package://${package}/meshes/manipulator/cyl.stl" scale="0.001 0.001 0.001"/>
+        <mesh filename="package://${package}/meshes/manipulators/5DOF/cyl.stl" scale="0.001 0.001 0.001"/>
       </geometry>
     </visual>
@@ -56,5 +56,5 @@
       <origin xyz="0 0 0" rpy="0 0 0" />
       <geometry>
-        <mesh filename="package://${package}/meshes/manipulator/arm1.stl" scale="0.001 0.001 0.001"/>
+        <mesh filename="package://${package}/meshes/manipulators/5DOF/arm1.stl" scale="0.001 0.001 0.001"/>
       </geometry>
     </visual>
@@ -75,5 +75,5 @@
       <origin xyz="0 0 0" rpy="0 0 0" />
       <geometry>
-        <mesh filename="package://${package}/meshes/manipulator/arm2.stl" scale="0.001 0.001 0.001"/>
+        <mesh filename="package://${package}/meshes/manipulators/5DOF/arm2.stl" scale="0.001 0.001 0.001"/>
       </geometry>
     </visual>
@@ -94,5 +94,5 @@
       <origin xyz="0 0 0" rpy="0 0 0" />
       <geometry>
-        <mesh filename="package://${package}/meshes/manipulator/arm3.stl" scale="0.001 0.001 0.001"/>
+        <mesh filename="package://${package}/meshes/manipulators/5DOF/arm3.stl" scale="0.001 0.001 0.001"/>
       </geometry>
     </visual>
@@ -116,5 +116,5 @@
       <origin xyz="0 0 0" rpy="0 0 0" />
       <geometry>
-        <mesh filename="package://${package}/meshes/manipulator/tool.stl" scale="0.001 0.001 0.001"/>
+        <mesh filename="package://${package}/meshes/manipulators/5DOF/tool.stl" scale="0.001 0.001 0.001"/>
       </geometry>
     </visual>
