Commit message: Updating code from rover

File: sirius_description/robots/sirius.urdf (robot description, URDF)
Before this commit: robot sirius, 30 links, 29 joints
Links:
- link back_left_inner_rim: geometry collision cylinder length=0.01 radius=0.08800000000000001; visual mesh filename=packa e://sirius_description/meshes/sirius/rim.stl scale=0.001 0.001 0.001

File: sirius_description/robots/sirius.urdf.xacro (robot description, xacro)
@@ -82,5 +82,6 @@
   <!-- Define subcomponents joints -->
   <xacro:joint child="platform"
-               xyz="0 0 ${mechanical['wheel_radius'] + mechanical['suspension_height'] - mechanical['suspension_z']}" />
+               xyz="0 0 ${mechanical['wheel_radius'] + mechanical['suspension_height'] - mechanical['suspension_z']}"
+               rpy="0 0 3.14"/>
   <xacro:joint parent="platform"
                child="back_left_suspension"
@@ -109,6 +110,6 @@
   <xacro:joint parent="platform"
                child="front_camera"
-               xyz="${mechanical['front_camera_xyz']}"
-               rpy="${mechanical['front_camera_rpy']}"/>
+               xyz="-0.574 0 0.936"
+               rpy="0 0.699 3.14"/>
   <xacro:joint parent="platform"  child="gnss" xyz="${mechanical['gnss_xyz']}" />
   <!-- Gazebo plugins -->
