Commit message: feat(sirius_gazebo): Provide gazebo origin coordinates to gnss plugin

File: sirius_description/robots/sirius.urdf.xacro (robot description, xacro)
@@ -6,4 +6,5 @@
   <xacro:arg name="elevation" default="0.0"/>
   <xacro:arg name="imu_frequency" default="200.0"/>
+  <xacro:arg name="gazebo_origin" default="[-9.39, 16.03]"/>
   <xacro:arg name="stereo_fps" default="30"/>
   <xacro:arg name="year" default=""/>
@@ -16,4 +17,5 @@
   <xacro:property name="elevation" value="$(arg elevation)" />
   <xacro:property name="imu_frequency" value="$(arg imu_frequency)" />
+  <xacro:property name="gazebo_origin" value="${$(arg gazebo_origin)}" />
   <xacro:property name="stereo_fps" value="$(arg stereo_fps)" />
   <xacro:property name="year" value="$(arg year)" />
@@ -123,4 +125,5 @@
       <topicName>ground_truth</topicName>
       <frameName>map</frameName>
+      <frameXyzOffset>${gazebo_origin[0]} ${gazebo_origin[1]} 0</frameXyzOffset>
       <frameRpyOffset>0 0 ${datum[2] * pi/180}</frameRpyOffset>
     </plugin>

File: sirius_description/urdf/sirius/gnss.urdf.xacro (robot description, xacro)
@@ -3,5 +3,5 @@
      https://www.sparkfun.com/products/21801 -->
 <robot xmlns:xacro="http://wiki.ros.org/xacro">
-<xacro:macro name="gnss" params="prefix:='' material collisions:=${xacro.load_yaml('$(find sirius_description)/urdf/sirius/collisions.yaml')} datum:=^ elevation:=^ horizontal_cep:=1.0 vertical_cep:=1.5 rate:=20.0">
+<xacro:macro name="gnss" params="prefix:='' material collisions:=${xacro.load_yaml('$(find sirius_description)/urdf/sirius/collisions.yaml')} datum:=^ elevation:=^ horizontal_cep:=1.0 vertical_cep:=1.5 rate:=20.0 spawn_origin:=^">
   <xacro:property name="_prefix" value="${prefix + '_' if prefix else ''}"/>
   <!-- sqrt(-1/(2*ln(0.5))) = 0.8493218002880191 -->
@@ -66,5 +66,6 @@
             <elevation>${elevation}</elevation>
         </sphericalCoordinates>
-        <positionCovariance>${horizontal_stddev} 0 0 0 ${horizontal_stddev} 0 0 0 ${vertical_stddev}</positionCovariance>
+        <!-- <positionCovariance>${horizontal_stddev} 0 0 0 ${horizontal_stddev} 0 0 0 ${vertical_stddev}</positionCovariance> -->
+        <spawnOrigin>${spawn_origin[0]} ${spawn_origin[1]}</spawnOrigin>
       </plugin>
     </sensor>

Commit message: Sirius simulation works in ROS2

File: sirius_description/robots/sirius.urdf.xacro (robot description, xacro)
@@ -75,8 +75,7 @@
   <xacro:joint parent="platform" child="front_camera" xyz="${mechanical['front_camera_xyz']}" rpy="${mechanical['front_camera_rpy']}"/>
   <xacro:joint parent="platform" child="gnss" xyz="${mechanical['gnss_xyz']}" />
-  <!--vvv TO DO: Adjust after implementing ros2_control and gazebo vvv-->
   <ros2_control name="GazeboSystem" type="system">
     <hardware>
-      <plugin>gazebo_ros2_control/GazeboSystem</plugin>
+      <plugin>gz_ros2_control/GazeboSimSystem</plugin>
     </hardware>
     <xacro:macro name="wheel_interface" params="name">
@@ -99,22 +98,16 @@
     <xacro:joint parent="platform" child="root_link" xyz="${mechanical['suspension_separation_x']/2} 0 ${mechanical['suspension_z'] + 0.045}" rpy="0 0 0"/>
   </xacro:if>
-  <gazebo>
-    <plugin filename="libgazebo_ros2_control.so" name="gazebo_ros2_control">
+<gazebo>
+    <!-- Plugin kontrolera -->
+    <plugin filename="gz_ros2_control-system" name="gz_ros2_control::GazeboSimROS2ControlPlugin">
       <parameters>$(find sirius_description)/config/controllers.yaml</parameters>
     </plugin>
-    <plugin name="p3d_plugin" filename="libgazebo_ros_p3d.so">
-      <ros>
-        <namespace>/</namespace>
-        <remapping>odom:=ground_truth</remapping>
-      </ros>
-      <always_on>true</always_on>
-      <update_rate>200.0</update_rate>
-      <body_name>base_link</body_name>
-      <frame_name>map</frame_name>
-      <xyz_offset>${gazebo_origin[0]} ${gazebo_origin[1]} 0</xyz_offset>
-      <rpy_offset>0 0 ${datum[2] * pi/180}</rpy_offset>
-      <gaussian_noise>0.0</gaussian_noise>
+    <!-- Plugin Odometrii -->
+    <plugin filename="gz-sim-odometry-publisher-system" name="gz::sim::systems::OdometryPublisher">
+      <odom_frame>map</odom_frame>
+      <robot_base_frame>base_link</robot_base_frame>
+      <odom_publish_frequency>200</odom_publish_frequency>
+      <odom_topic>ground_truth</odom_topic>
     </plugin>
   </gazebo>
-  <!--^^^ TO DO: Adjust after implementing ros2_control and gazebo ^^^-->
 </robot>

File: sirius_description/urdf/hp_4310/hp_4310.urdf.xacro (robot description, xacro)
@@ -16,5 +16,5 @@
     </collision>
   </link>
-  <gazebo reference="${prefix}_camera">
+  <!-- <gazebo reference="${prefix}_camera">
       <visual>
         <xacro:element xacro:name="xacro:${material}" />
@@ -54,5 +54,5 @@
       </plugin>
     </sensor>
-  </gazebo>
+  </gazebo> -->
 </xacro:macro>
 </robot>

File: sirius_description/urdf/oak-d-w/oak-d-w.urdf.xacro (robot description, xacro)
@@ -67,10 +67,11 @@
   </joint>
   <gazebo reference="${prefix}_right_camera_optical">
-    <sensor type="multicamera" name="${prefix}_stereo_camera">
-      <always_on>true</always_on>
+    <sensor type="camera" name="${prefix}_left">
+      <visualize>true</visualize>
       <update_rate>${stereo_fps}</update_rate>
-      <visualize>false</visualize>
-      <camera name="left">
-        <pose>${calibration.cam1.T_cn_cnm1[0][3]} ${calibration.cam1.T_cn_cnm1[1][3]} ${calibration.cam1.T_cn_cnm1[2][3] - optical_offset_x} ${atan2(calibration.cam1.T_cn_cnm1[2][1],calibration.cam1.T_cn_cnm1[2][2]) + pi/2} ${atan2(-calibration.cam1.T_cn_cnm1[2][0],sqrt(calibration.cam1.T_cn_cnm1[2][1]**2 + calibration.cam1.T_cn_cnm1[2][2]**2)) - pi/2} ${atan2(calibration.cam1.T_cn_cnm1[1][0],calibration.cam1.T_cn_cnm1[0][0])}</pose>
+      <topic>${prefix}/left/image_raw</topic>
+      <gz_frame_id>${prefix}_left_camera_optical</gz_frame_id>
+      <pose>${calibration.cam1.T_cn_cnm1[0][3]} ${calibration.cam1.T_cn_cnm1[1][3]} ${calibration.cam1.T_cn_cnm1[2][3] - optical_offset_x} ${atan2(calibration.cam1.T_cn_cnm1[2][1],calibration.cam1.T_cn_cnm1[2][2]) + pi/2} ${atan2(-calibration.cam1.T_cn_cnm1[2][0],sqrt(calibration.cam1.T_cn_cnm1[2][1]**2 + calibration.cam1.T_cn_cnm1[2][2]**2)) - pi/2} ${atan2(calibration.cam1.T_cn_cnm1[1][0],calibration.cam1.T_cn_cnm1[0][0])}</pose>
+      <camera>
         <horizontal_fov>${2*atan2(calibration.cam0.resolution[0], calibration.cam0.intrinsics[0] + calibration.cam0.intrinsics[1])}</horizontal_fov>
         <image>
@@ -80,15 +81,16 @@
         </image>
         <clip>
-          <near>0.02</near>
-          <far>300</far>
+          <near>0.1</near>
+          <far>100</far>
         </clip>
-        <noise>
-          <type>gaussian</type>
-          <mean>0.0</mean>
-          <stddev>0.007</stddev>
-        </noise>
       </camera>
-      <camera name="right">
-        <pose>0 0 ${-optical_offset_x} ${pi/2} ${-pi/2} 0</pose>
+    </sensor>
+    <sensor type="camera" name="${prefix}_right">
+      <visualize>true</visualize>
+      <update_rate>${stereo_fps}</update_rate>
+      <topic>${prefix}/right/image_raw</topic>
+      <gz_frame_id>${prefix}_right_camera_optical</gz_frame_id>
+      <pose>0 0 ${-optical_offset_x} ${pi/2} ${-pi/2} 0</pose>
+      <camera>
         <horizontal_fov>${2*atan2(calibration.cam0.resolution[0], calibration.cam0.intrinsics[0] + calibration.cam0.intrinsics[1])}</horizontal_fov>
         <image>
@@ -98,7 +100,51 @@
         </image>
         <clip>
+          <near>0.1</near>
+          <far>100</far>
+        </clip>
+      </camera>
+    </sensor>
+  </gazebo>
+  <gazebo reference="${prefix}_camera">
+    <sensor name="${prefix}_camera" type="rgbd_camera">
+      <topic>${prefix}/camera</topic>
+      <gz_frame_id>${prefix}_camera</gz_frame_id>
+      <pose>0 0 0 0 0 0</pose>
+      <always_on>1</always_on>
+      <update_rate>${stereo_fps}</update_rate>
+      <camera name="${prefix}_camera_depth">
+        <horizontal_fov>${2*atan2(calibration.cam0.resolution[0], calibration.cam0.intrinsics[0] + calibration.cam0.intrinsics[1])}</horizontal_fov>
+        <image>
+          <width>${calibration.cam0.resolution[0]}</width>
+          <height>${calibration.cam0.resolution[1]}</height>
+          <format>R8G8B8</format>
+        </image>
+        <lens>
+          <intrinsics>
+            <fx>${calibration.cam0.intrinsics[0]}</fx>
+            <fy>${calibration.cam0.intrinsics[1]}</fy>
+            <cx>${calibration.cam0.intrinsics[2]}</cx>
+            <cy>${calibration.cam0.intrinsics[3]}</cy>
+            <s>0</s>
+          </intrinsics>
+        </lens>
+        <distortion>
+          <k1>${calibration.cam0.distortion_coeffs[0]}</k1>
+          <k2>${calibration.cam0.distortion_coeffs[1]}</k2>
+          <k3>${calibration.cam0.distortion_coeffs[2]}</k3>
+          <p1>${calibration.cam0.distortion_coeffs[3]}</p1>
+          <p2>0.0</p2>
+          <center>0.5 0.5</center>
+        </distortion>
+        <clip>
           <near>0.02</near>
           <far>300</far>
         </clip>
+        <depth_camera>
+          <clip>
+            <near>0.35</near>
+            <far>35.0</far>
+          </clip>
+        </depth_camera>
         <noise>
           <type>gaussian</type>
@@ -107,78 +153,35 @@
         </noise>
       </camera>
-      <plugin name="stereo_camera_controller" filename="libgazebo_ros_camera.so">
-        <ros>
-          <namespace>/${prefix}_camera</namespace>
-          <remapping>left/image_raw:=image_rect</remapping>
-          <remapping>right/image_raw:=right/image_rect</remapping>
-          <remapping>left/camera_info:=camera_info</remapping>
-          <remapping>right/camera_info:=right/camera_info</remapping>
-        </ros>
-        <camera_name>stereo</camera_name>
-        <frame_name>${prefix}_left_camera_optical</frame_name>
-        <hack_baseline>${baseline}</hack_baseline>
-      </plugin>
-    </sensor>
-  </gazebo>
-  <gazebo reference="${prefix}_camera">
-    <sensor type="depth" name="${prefix}_camera_depth">
-      <always_on>true</always_on>
-      <update_rate>${stereo_fps}</update_rate>
-      <visualize>false</visualize>
-      <camera name="depth_cam">
-        <horizontal_fov>${2*atan2(calibration.cam0.resolution[0], calibration.cam0.intrinsics[0] + calibration.cam0.intrinsics[1])}</horizontal_fov>
-        <image>
-          <width>${calibration.cam0.resolution[0]}</width>
-          <height>${calibration.cam0.resolution[1]}</height>
-          <format>R8G8B8</format>
-        </image>
-        <clip>
-          <near>0.02</near>
-          <far>300</far>
-        </clip>
-        <noise>
-          <type>gaussian</type>
-          <mean>0.0</mean>
-          <stddev>0.007</stddev>
-        </noise>
-      </camera>
-      <plugin name="camera_controller" filename="libgazebo_ros_camera.so">
-        <ros>
-          <namespace>/${prefix}_camera</namespace>
-          <remapping>custom_cam/image_raw:=rgb/image_rect_color</remapping>
-          <remapping>custom_cam/camera_info:=rgb/camera_info</remapping>
-          <remapping>custom_cam/depth/image_raw:=depth_registered/image</remapping>
-          <remapping>custom_cam/points:=depth_registered/points</remapping>
-        </ros>
-        <camera_name>rgb</camera_name>
-        <frame_name>${prefix}_rgb_camera_optical</frame_name>
-        <hack_baseline>0.0</hack_baseline>
-        <min_depth>0.35</min_depth>
-        <max_depth>35.0</max_depth>
-      </plugin>
-    </sensor>
-  </gazebo>
-  <gazebo reference="${prefix}_camera_imu_link">
-    <sensor type="imu" name="imu_sensor">
-      <always_on>true</always_on>
+    </sensor>
+  </gazebo>
+<gazebo reference="${prefix}_camera_imu_link">
+    <sensor name="${prefix}_imu_sensor" type="imu">
+      <always_on>1</always_on>
       <update_rate>${imu_frequency}</update_rate>
+      <topic>${prefix}/imu/data</topic>
+      <gz_frame_id>${prefix}_camera_imu_link</gz_frame_id>
       <imu>
+        <!-- Wyłączamy orientację, jeśli ma być liczona przez zewnętrzny filtr (np. EKF) -->
+        <enable_orientation>0</enable_orientation>
         <angular_velocity>
           <x>
             <noise type="gaussian">
+              <mean>0</mean>
               <stddev>${gyroscope_stddev}</stddev>
-              <bias_stddev>${gyroscope_bias_stddev}</bias_stddev>
+              <dynamic_bias_stddev>${gyroscope_bias_stddev}</dynamic_bias_stddev>
             </noise>
           </x>
           <y>
             <noise type="gaussian">
+              <mean>0</mean>
               <stddev>${gyroscope_stddev}</stddev>
-              <bias_stddev>${gyroscope_bias_stddev}</bias_stddev>
+              <dynamic_bias_stddev>${gyroscope_bias_stddev}</dynamic_bias_stddev>
             </noise>
           </y>
           <z>
             <noise type="gaussian">
+              <mean>0</mean>
               <stddev>${gyroscope_stddev}</stddev>
-              <bias_stddev>${gyroscope_bias_stddev}</bias_stddev>
+              <dynamic_bias_stddev>${gyroscope_bias_stddev}</dynamic_bias_stddev>
             </noise>
           </z>
@@ -187,31 +190,25 @@
           <x>
             <noise type="gaussian">
+              <mean>0</mean>
               <stddev>${accelerometer_stddev}</stddev>
-              <bias_stddev>${accelerometer_bias_stddev}</bias_stddev>
+              <dynamic_bias_stddev>${accelerometer_bias_stddev}</dynamic_bias_stddev>
             </noise>
           </x>
           <y>
             <noise type="gaussian">
+              <mean>0</mean>
               <stddev>${accelerometer_stddev}</stddev>
-              <bias_stddev>${accelerometer_bias_stddev}</bias_stddev>
+              <dynamic_bias_stddev>${accelerometer_bias_stddev}</dynamic_bias_stddev>
             </noise>
           </y>
           <z>
             <noise type="gaussian">
+              <mean>0</mean>
               <stddev>${accelerometer_stddev}</stddev>
-              <bias_stddev>${accelerometer_bias_stddev}</bias_stddev>
+              <dynamic_bias_stddev>${accelerometer_bias_stddev}</dynamic_bias_stddev>
             </noise>
           </z>
         </linear_acceleration>
       </imu>
-      <!-- Zamiana libsirius... na standardowy plugin -->
-      <plugin filename="libgazebo_ros_imu_sensor.so" name="imu_plugin">
-        <ros>
-            <namespace>/${prefix}_camera/imu</namespace>
-            <remapping>~/out:=data</remapping>
-        </ros>
-        <frame_name>${prefix}_camera_imu_link</frame_name>
-        <initial_orientation_as_reference>false</initial_orientation_as_reference>
-      </plugin>
     </sensor>
   </gazebo>
@@ -237,5 +234,5 @@
         </z>
       </magnetometer>
-      <plugin filename="libgazebo_ros_magnetometer_sensor.so" name="magnetometer_plugin">
+      <!-- <plugin filename="libgazebo_ros_magnetometer_sensor.so" name="magnetometer_plugin">
         <ros>
             <namespace>/${prefix}_camera/imu</namespace>
@@ -243,5 +240,5 @@
         </ros>
         <frame_name>${prefix}_camera_imu_link</frame_name>
-      </plugin>
+      </plugin> -->
     </sensor>
   </gazebo>

File: sirius_description/urdf/sirius/gnss.urdf.xacro (robot description, xacro)
@@ -56,5 +56,5 @@
         </velocity_sensing>
       </gps>
-      <plugin filename="libsirius_gazebo_ros_gps_sensor.so" name="gps_plugin">
+      <!-- <plugin filename="libsirius_gazebo_ros_gps_sensor.so" name="gps_plugin">
         <topicName>/gps/fix</topicName>
         <frameName>gnss</frameName>
@@ -68,5 +68,5 @@
         <positionCovariance>${horizontal_stddev} 0 0 0 ${horizontal_stddev} 0 0 0 ${vertical_stddev}</positionCovariance>
         <gazeboOrigin>${gazebo_origin[0]} ${gazebo_origin[1]}</gazeboOrigin>
-      </plugin>
+      </plugin> -->
     </sensor>
   </gazebo>

File: sirius_description/urdf/sirius/manipulators/5DOF.urdf.xacro (robot description, xacro)
@@ -122,8 +122,8 @@
   <link name="virtual">
   </link>
-    <joint name="tool_virtual" type="fixed">
-      <parent link="tool"/>
-      <child link="virtual"/>
-      <origin xyz="0 0 ${tool_length}"/>
-    </joint>
+  <joint name="tool_virtual" type="fixed">
+    <parent link="tool"/>
+    <child link="virtual"/>
+    <origin xyz="0 0 ${tool_length}"/>
+  </joint>
 </robot>
