Commit message: Migration of ROS1 sirius rover packages - changes to be chacked

File: sirius_description/robots/sirius.urdf.xacro (robot description, xacro)
@@ -9,4 +9,6 @@
   <xacro:arg name="year" default=""/>
   <xacro:arg name="manipulator" default="none"/>
+  <!-- Set to 'true' to use real hardware interfaces instead of Gazebo simulation -->
+  <xacro:arg name="use_real_hardware" default="false"/>
   <xacro:property name="calibration_path" value="$(arg calibration_path)" />
   <xacro:if value="${calibration_path != ''}">
@@ -75,7 +77,20 @@
   <xacro:joint parent="platform" child="front_camera" xyz="${mechanical['front_camera_xyz']}" rpy="${mechanical['front_camera_rpy']}"/>
   <xacro:joint parent="platform" child="gnss" xyz="${mechanical['gnss_xyz']}" />
-  <ros2_control name="GazeboSystem" type="system">
+  <!-- ================================================================
+       Wheel drive system — switches between real hardware and Gazebo.
+       ================================================================ -->
+  <xacro:property name="use_real_hardware" value="$(arg use_real_hardware)"/>
+  <ros2_control name="SiriusWheelSystem" type="system">
     <hardware>
-      <plugin>gz_ros2_control/GazeboSimSystem</plugin>
+      <xacro:if value="${use_real_hardware}">
+        <!-- ODrive topic-bridge plugin (communicates via relaxing_middleware) -->
+        <plugin>sirius_hw_interfaces/SiriusWheelsHW</plugin>
+        <param name="driver_namespaces">
+          /wheels_left/motor0,/wheels_left/motor1,/wheels_right/motor0,/wheels_right/motor1
+        </param>
+      </xacro:if>
+      <xacro:unless value="${use_real_hardware}">
+        <plugin>gz_ros2_control/GazeboSimSystem</plugin>
+      </xacro:unless>
     </hardware>
     <xacro:macro name="wheel_interface" params="name">
@@ -87,4 +102,5 @@
         <state_interface name="velocity"/>
         <state_interface name="position"/>
+        <state_interface name="effort"/>
       </joint>
     </xacro:macro>
@@ -97,4 +113,111 @@
     <xacro:include filename="$(find sirius_description)/urdf/sirius/manipulators/$(arg manipulator).urdf.xacro" />
     <xacro:joint parent="platform" child="root_link" xyz="${mechanical['suspension_separation_x']/2} 0 ${mechanical['suspension_z'] + 0.045}" rpy="0 0 0"/>
+    <!-- Manipulator ros2_control system — real or simulated -->
+    <xacro:if value="${manipulator == '5DOF'}">
+      <ros2_control name="SiriusManipSystem" type="system">
+        <hardware>
+          <xacro:if value="${use_real_hardware}">
+            <plugin>sirius_hw_interfaces/SiriusManipHW</plugin>
+            <param name="state_topic">/manip/joint_states</param>
+            <param name="command_topic">/manip/set_joint_states</param>
+          </xacro:if>
+          <xacro:unless value="${use_real_hardware}">
+            <plugin>gz_ros2_control/GazeboSimSystem</plugin>
+          </xacro:unless>
+        </hardware>
+        <joint name="waist">
+          <command_interface name="position"/>
+          <command_interface name="velocity"/>
+          <command_interface name="effort"/>
+          <state_interface name="position"><param name="initial_value">0.0</param></state_interface>
+          <state_interface name="velocity"/>
+          <state_interface name="effort"/>
+        </joint>
+        <joint name="shoulder">
+          <command_interface name="position"/>
+          <command_interface name="velocity"/>
+          <command_interface name="effort"/>
+          <state_interface name="position"><param name="initial_value">0.0</param></state_interface>
+          <state_interface name="velocity"/>
+          <state_interface name="effort"/>
+        </joint>
+        <joint name="elbow">
+          <command_interface name="position"/>
+          <command_interface name="velocity"/>
+          <command_interface name="effort"/>
+          <state_interface name="position"><param name="initial_value">0.0</param></state_interface>
+          <state_interface name="velocity"/>
+          <state_interface name="effort"/>
+        </joint>
+        <joint name="wrist_lift">
+          <command_interface name="position"/>
+          <command_interface name="velocity"/>
+          <command_interface name="effort"/>
+          <state_interface name="position"><param name="initial_value">0.0</param></state_interface>
+          <state_interface name="velocity"/>
+          <state_interface name="effort"/>
+        </joint>
+        <joint name="wrist_turn">
+          <command_interface name="position"/>
+          <command_interface name="velocity"/>
+          <command_interface name="effort"/>
+          <state_interface name="position"><param name="initial_value">0.0</param></state_interface>
+          <state_interface name="velocity"/>
+          <state_interface name="effort"/>
+        </joint>
+        <joint name="wrist_spin">
+          <command_interface name="position"/>
+          <command_interface name="velocity"/>
+          <command_interface name="effort"/>
+          <state_interface name="position"><param name="initial_value">0.0</param></state_interface>
+          <state_interface name="velocity"/>
+          <state_interface name="effort"/>
+        </joint>
+      </ros2_control>
+    </xacro:if>
+    <xacro:if value="${manipulator == '6DOF'}">
+      <ros2_control name="SiriusManipSystem" type="system">
+        <hardware>
+          <xacro:if value="${use_real_hardware}">
+            <plugin>sirius_hw_interfaces/SiriusManipHW</plugin>
+            <param name="state_topic">/manip/joint_states</param>
+            <param name="command_topic">/manip/set_joint_states</param>
+          </xacro:if>
+          <xacro:unless value="${use_real_hardware}">
+            <plugin>gz_ros2_control/GazeboSimSystem</plugin>
+          </xacro:unless>
+        </hardware>
+        <joint name="joint_1">
+          <command_interface name="position"/>
+          <state_interface name="position"><param name="initial_value">0.0</param></state_interface>
+          <state_interface name="velocity"/>
+        </joint>
+        <joint name="joint_2">
+          <command_interface name="position"/>
+          <state_interface name="position"><param name="initial_value">0.0</param></state_interface>
+          <state_interface name="velocity"/>
+        </joint>
+        <joint name="joint_3">
+          <command_interface name="position"/>
+          <state_interface name="position"><param name="initial_value">0.0</param></state_interface>
+          <state_interface name="velocity"/>
+        </joint>
+        <joint name="joint_4">
+          <command_interface name="position"/>
+          <state_interface name="position"><param name="initial_value">0.0</param></state_interface>
+          <state_interface name="velocity"/>
+        </joint>
+        <joint name="joint_5">
+          <command_interface name="position"/>
+          <state_interface name="position"><param name="initial_value">0.0</param></state_interface>
+          <state_interface name="velocity"/>
+        </joint>
+        <joint name="joint_6">
+          <command_interface name="position"/>
+          <state_interface name="position"><param name="initial_value">0.0</param></state_interface>
+          <state_interface name="velocity"/>
+        </joint>
+      </ros2_control>
+    </xacro:if>
   </xacro:if>
 <gazebo>

File: sirius_description/urdf/sirius/manipulators/5DOF.urdf.xacro (robot description, xacro)
@@ -13,4 +13,13 @@
   <xacro:property name="arm2_home_angle" value="2.356194490192345"/>
   <xacro:property name="arm3_home_angle" value="0.5"/>
+  <!-- Minimal inertia for Gazebo simulation — physically plausible box estimates. -->
+  <xacro:macro name="box_inertia" params="m x y z">
+    <inertial>
+      <mass value="${m}"/>
+      <inertia ixx="${m*(y*y+z*z)/12}" ixy="0" ixz="0"
+               iyy="${m*(x*x+z*z)/12}" iyz="0"
+               izz="${m*(x*x+y*y)/12}"/>
+    </inertial>
+  </xacro:macro>
   <link name="root_link">
   </link>
@@ -26,4 +35,5 @@
       </geometry>
     </visual>
+    <xacro:box_inertia m="0.5" x="0.20" y="0.20" z="0.06"/>
   </link>
   <joint name="waist" type="continuous">
@@ -40,4 +50,5 @@
       </geometry>
     </visual>
+    <xacro:box_inertia m="0.2" x="0.08" y="0.08" z="${cyl_length}"/>
   </link>
   <joint name="shoulder" type="revolute">
@@ -59,4 +70,5 @@
       </geometry>
     </visual>
+    <xacro:box_inertia m="0.8" x="0.05" y="0.05" z="${arm1_length}"/>
   </link>
   <joint name="elbow" type="revolute">
@@ -78,4 +90,5 @@
       </geometry>
     </visual>
+    <xacro:box_inertia m="0.6" x="0.05" y="0.05" z="${arm2_length}"/>
   </link>
   <joint name="wrist_lift" type="revolute">
@@ -97,4 +110,5 @@
       </geometry>
     </visual>
+    <xacro:box_inertia m="0.2" x="0.05" y="0.05" z="${arm3_length}"/>
   </link>
   <joint name="wrist_turn" type="continuous">
@@ -105,4 +119,5 @@
   </joint>
   <link name="fake">
+    <xacro:box_inertia m="0.01" x="0.02" y="0.02" z="0.02"/>
   </link>
   <joint name="wrist_spin" type="continuous">
@@ -119,4 +134,5 @@
       </geometry>
     </visual>
+    <xacro:box_inertia m="0.3" x="0.10" y="0.10" z="${tool_length}"/>
   </link>
   <link name="virtual">

File: sirius_description/urdf/sirius/manipulators/6DOF.urdf.xacro (robot description, xacro)
@@ -8,5 +8,4 @@
     <visual>
       <geometry>
-        <!-- <cylinder length="0.05" radius="0.1"/> -->
         <mesh filename="package://sirius_description/meshes/manipulators/6DOF/global_roll_assembly.STL" scale="0.001 0.001 0.001"/>
       </geometry>
@@ -18,9 +17,12 @@
     <collision>
       <geometry>
-          <!-- <cylinder length="0.05" radius="0.1"/> -->
           <mesh filename="package://sirius_description/meshes/manipulators/6DOF/global_roll_assembly.STL" scale="0.001 0.001 0.001"/>
       </geometry>
       <origin xyz="0.0 0.0 0.1" rpy="0.0 0.0 0.0"/>
     </collision>
+    <inertial>
+      <mass value="0.5"/>
+      <inertia ixx="0.0042" ixy="0" ixz="0" iyy="0.0042" iyz="0" izz="0.0025"/>
+    </inertial>
   </link>
   <!-- Joints and links -->
@@ -28,8 +30,6 @@
     <visual>
       <geometry>
-        <!-- <cylinder length="0.1" radius="0.05"/> -->
         <mesh filename="package://sirius_description/meshes/manipulators/6DOF/base_assy.STL" scale="0.001 0.001 0.001"/>
       </geometry>
-      <!-- <origin xyz="-0.6 -0.2 -0.022" rpy="0.0 0.0 0.0"/> -->
       <origin xyz="0.0 0.0 0.0" rpy="0.0 0.0 0.0"/>
       <material name="purple">
@@ -39,10 +39,12 @@
     <collision>
       <geometry>
-          <!-- <cylinder length="0.1" radius="0.05"/> -->
           <mesh filename="package://sirius_description/meshes/manipulators/6DOF/base_assy.STL" scale="0.001 0.001 0.001"/>
       </geometry>
-      <!-- <origin xyz="-0.1 -0.1 -0.022" rpy="0.0 0.0 0.0"/> -->
-      <origin xyz="0.0 0.0 0.0" rpy="0.0 0.0 0.0"/>
-    </collision>
+      <origin xyz="0.0 0.0 0.0" rpy="0.0 0.0 0.0"/>
+    </collision>
+    <inertial>
+      <mass value="0.8"/>
+      <inertia ixx="0.0034" ixy="0" ixz="0" iyy="0.0034" iyz="0" izz="0.0016"/>
+    </inertial>
   </link>
   <joint name="joint_1" type="revolute">
@@ -57,5 +59,4 @@
       <geometry>
         <mesh filename="package://sirius_description/meshes/manipulators/6DOF/GP1.STL" scale="0.001 0.001 0.001"/>
-        <!-- <cylinder length="0.46" radius="0.05"/> -->
       </geometry>
       <origin xyz="0 0 0" rpy="0.0 0.0 0.0"/>
@@ -67,8 +68,11 @@
       <geometry>
         <mesh filename="package://sirius_description/meshes/manipulators/6DOF/GP1.STL" scale="0.001 0.001 0.001"/>
-        <!-- <cylinder length="0.46" radius="0.05"/> -->
-      </geometry>
-      <origin xyz="0 0 0" rpy="0.0 0.0 0.0"/>
-    </collision>
+      </geometry>
+      <origin xyz="0 0 0" rpy="0.0 0.0 0.0"/>
+    </collision>
+    <inertial>
+      <mass value="1.2"/>
+      <inertia ixx="0.024" ixy="0" ixz="0" iyy="0.024" iyz="0" izz="0.0024"/>
+    </inertial>
   </link>
   <joint name="joint_2" type="revolute">
@@ -83,5 +87,4 @@
     <visual>
       <geometry>
-        <!-- <cylinder length="0.340" radius="0.05"/> -->
         <mesh filename="package://sirius_description/meshes/manipulators/6DOF/GP2.STL" scale="0.001 0.001 0.001"/>
       </geometry>
@@ -93,9 +96,12 @@
     <collision>
       <geometry>
-          <!-- <cylinder length="0.680" radius="0.05"/> -->
           <mesh filename="package://sirius_description/meshes/manipulators/6DOF/GP2.STL" scale="0.001 0.001 0.001"/>
       </geometry>
       <origin xyz="0 0 0" rpy="0.0 0.0 0.0"/>
     </collision>
+    <inertial>
+      <mass value="0.8"/>
+      <inertia ixx="0.012" ixy="0" ixz="0" iyy="0.012" iyz="0" izz="0.0016"/>
+    </inertial>
   </link>
   <joint name="joint_3" type="revolute">
@@ -109,5 +115,4 @@
     <visual>
       <geometry>
-        <!-- <cylinder length="0.07" radius="0.04"/> -->
         <mesh filename="package://sirius_description/meshes/manipulators/6DOF/wrist_diff_base.STL" scale="0.001 0.001 0.001"/>
       </geometry>
@@ -119,9 +124,12 @@
     <collision>
       <geometry>
-          <!-- <cylinder length="0.07" radius="0.05"/> -->
           <mesh filename="package://sirius_description/meshes/manipulators/6DOF/wrist_diff_base.STL" scale="0.001 0.001 0.001"/>
       </geometry>
       <origin xyz="0.0 0.0 0.0" rpy="0.0 0.0 0.0"/>
     </collision>
+    <inertial>
+      <mass value="0.3"/>
+      <inertia ixx="0.0005" ixy="0" ixz="0" iyy="0.0005" iyz="0" izz="0.0003"/>
+    </inertial>
   </link>
   <joint name="joint_4" type="revolute">
@@ -135,5 +143,4 @@
     <visual>
       <geometry>
-        <!-- <box size="0.03 0.150 0.03"/> -->
         <mesh filename="package://sirius_description/meshes/manipulators/6DOF/wrist_diff_output.STL" scale="0.001 0.001 0.001"/>
       </geometry>
@@ -145,9 +152,12 @@
     <collision>
       <geometry>
-        <!-- <box size="0.03 0.150 0.03"/>       -->
         <mesh filename="package://sirius_description/meshes/manipulators/6DOF/wrist_diff_output.STL" scale="0.001 0.001 0.001"/>
       </geometry>
       <origin xyz="0.0 0.0 0.0" rpy="0.0 0.0 0.0"/>
     </collision>
+    <inertial>
+      <mass value="0.2"/>
+      <inertia ixx="0.0007" ixy="0" ixz="0" iyy="0.0001" iyz="0" izz="0.0007"/>
+    </inertial>
   </link>
   <joint name="joint_5" type="revolute">
@@ -161,5 +171,4 @@
     <visual>
       <geometry>
-        <!-- <box size="0.01 0.01 0.1"/> -->
         <mesh filename="package://sirius_description/meshes/manipulators/6DOF/gripper.STL" scale="0.001 0.001 0.001"/>
       </geometry>
@@ -175,4 +184,8 @@
       <origin xyz="0.0 0.0 0.0" rpy="0.0 0.0 0.0"/>
     </collision>
+    <inertial>
+      <mass value="0.3"/>
+      <inertia ixx="0.0003" ixy="0" ixz="0" iyy="0.0003" iyz="0" izz="0.0002"/>
+    </inertial>
   </link>
   <joint name="joint_6" type="revolute">
