Commit message: Add gripper and fix joint control directions

File: manip/urdf/sirius2_manip.urdf.xacro (robot description, xacro)
@@ -153,5 +153,5 @@
     <parent link="link4"/>
     <child link="link5"/>
-    <axis xyz="0 -1 0"/>
+    <axis xyz="0 1 0"/>
     <limit lower="-1.55" upper="1.55" effort="1000.0" velocity="0.5"/>
     <origin xyz="0 0 0.07825 " rpy="0.0 0 0"/>

Commit message: random changes from the last year

File: manip/urdf/sirius2_manip.urdf.xacro (robot description, xacro)
@@ -108,5 +108,5 @@
         <mesh filename="package://manip/meshes/gripper.STL" scale="0.001 0.001 0.001"/>
       </geometry>
-      <origin xyz="0.0 0.0 0.0" rpy="0.0 0.0 0.0"/>
+      <origin xyz="0.0 0.0 0.0" rpy="0.0 0.0 1.5708"/>
       <material name="pink">
         <color rgba="0.0 0.0 1.0 1.0"/>
@@ -117,8 +117,9 @@
         <mesh filename="package://manip/meshes/gripper.STL" scale="0.001 0.001 0.001"/>
       </geometry>
-      <origin xyz="0.0 0.0 0.0" rpy="0.0 0.0 0.0"/>
+      <origin xyz="0.0 0.0 0.0" rpy="0.0 0.0 1.5708"/>
     </collision>
   </link>
   <link name="tool"/>
+  <link name="wrist_camera"/>
   <joint name="joint1" type="revolute">
     <parent link="base_link"/>
@@ -165,7 +166,12 @@
   </joint>
   <joint name="link6_to_tool" type="fixed">
-    <origin xyz="0 0 0.12" rpy="1.5708 -1.5708 0"/>
+    <origin xyz="0 0 0.12" rpy="0 0 0"/>
     <parent link="link6"/>
     <child link="tool"/>
   </joint>
+  <joint name="link5_to_wrist_camera" type="fixed">
+    <origin xyz="0 0.09 0.035" rpy="1.5708 -1.4 -1.5708"/>
+    <parent link="link5"/>
+    <child link="wrist_camera"/>
+  </joint>
 </robot>

Commit message: Current verion of soft

File: manip/urdf/sirius2_manip.urdf.xacro (robot description, xacro)
@@ -170,7 +170,12 @@
     <child link="tool"/>
   </joint>
-  <joint name="link5_to_wrist_camera" type="fixed">
-    <origin xyz="0 0.09 0.035" rpy="1.5708 -1.4 -1.5708"/>
+  <!-- <joint name="link6_to_wrist_camera" type="fixed">
+    <origin xyz="0 0.145 0.100" rpy="1.5708 -0.785398 -1.5708"/>
     <parent link="link5"/>
+    <child link="wrist_camera"/>
+  </joint> -->
+  <joint name="link6_to_wrist_camera" type="fixed">
+    <origin xyz="0 0 0.1" rpy="1.5708 -1.5708 0"/>
+    <parent link="link6"/>
     <child link="wrist_camera"/>
   </joint>
